File: pcb/ChakraPendant.sch (EAGLE design)
At the start: 19 parts, among them Q1 MOSFET-NCHANNEL2N7002PW

Commit message: WHO THE HELL KNOWS?
Parts:
- removed Q1: MOSFET-NCHANNEL2N7002PW, SparkFun-DiscreteSemi:MOSFET-NCHANNEL2N7002PW
- removed R4: 220, SparkFun-Passives:RESISTOR0603-RES
- added C4: 1uF, SparkFun-Passives:CAP0603-CAP
- added C5: 0.1uF, SparkFun-Passives:CAP0603-CAP
- added LEDSW: (no value), IC:ETA3406
Connections:
- removed net N$1: Q1.G, R4.2
- removed net N$2: C3.2, LEDPWR.2, Q1.D
- new net N$6: C3.1, C5.1, LEDPWR.1, LEDSW.EN
- new net STAT: CHARGE.STAT, LED2.A
- net +4.1V: now also C4.1, LEDSW.FB; no longer C3.1, LEDPWR.1
- net GND: now also C3.2, C4.2, C5.2, LEDPWR.2, LEDSW.GND; no longer Q1.S
- net PB2-SCK: now also LEDSW.IN; no longer R4.1
- net PB3-ADC3: no longer CHARGE.STAT, LED2.A
Other:
- moved on the sheet: C3, LEDPWR
Changed lines of the file:
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@@
 <layer number="223" name="223bmp" color="24" fill="1" visible="no" active="no"/>
 <layer number="224" name="224bmp" color="25" fill="1" visible="no" active="no"/>
+<layer number="225" name="225bmp" color="7" fill="1" visible="no" active="yes"/>
+<layer number="226" name="226bmp" color="7" fill="1" visible="no" active="yes"/>
+<layer number="227" name="227bmp" color="7" fill="1" visible="no" active="yes"/>
+<layer number="228" name="228bmp" color="7" fill="1" visible="no" active="yes"/>
+<layer number="230" name="230bmp" color="7" fill="1" visible="no" active="yes"/>
 <layer number="248" name="Housing" color="7" fill="1" visible="yes" active="yes"/>
 <layer number="249" name="Edge" color="7" fill="1" visible="yes" active="yes"/>
@@
 <part name="C2" library="SparkFun-Passives" deviceset="CAP" device="0603-CAP" value="4.7 uF"/>
 <part name="C3" library="SparkFun-Passives" deviceset="CAP" device="1206" value="22 uF"/>
-<part name="Q1" library="SparkFun-DiscreteSemi" deviceset="MOSFET-NCHANNEL" device="2N7002PW"/>
 <part name="U$1" library="Protofusion" deviceset="POGOPIN-CONN" device="WITHVIAS"/>
 <part name="S2" library="SparkFun-Electromechanical" deviceset="SWITCH-MOMENTARY-2" device="SMD-3"/>
@@
 <part name="SUPPLY1" library="supply2" deviceset="GND" device=""/>
 <part name="FRAME1" library="SparkFun-Aesthetics" deviceset="FRAME-LETTER" device=""/>
-<part name="R4" library="SparkFun-Passives" deviceset="RESISTOR" device="0603-RES" value="220"/>
+<part name="LEDSW" library="IC" deviceset="ETA3406" device=""/>
+<part name="SUPPLY3" library="supply2" deviceset="GND" device=""/>
+<part name="C4" library="SparkFun-Passives" deviceset="CAP" device="0603-CAP" value="1uF"/>
+<part name="SUPPLY4" library="supply2" deviceset="GND" device=""/>
+<part name="C5" library="SparkFun-Passives" deviceset="CAP" device="0603-CAP" value="0.1uF"/>
+<part name="SUPPLY14" library="supply2" deviceset="GND" device=""/>
 </parts>
 <sheets>
@@
 <instance part="JP1" gate="G$1" x="12.7" y="154.94" rot="MR90"/>
 <instance part="SUPPLY2" gate="GND" x="15.24" y="68.58"/>
-<instance part="SUPPLY5" gate="GND" x="121.92" y="71.12"/>
+<instance part="SUPPLY5" gate="GND" x="121.92" y="40.64"/>
 <instance part="SUPPLY6" gate="GND" x="91.44" y="86.36"/>
 <instance part="SUPPLY9" gate="GND" x="60.96" y="27.94"/>
@@
 <instance part="C1" gate="G$1" x="15.24" y="127" rot="MR0"/>
 <instance part="C2" gate="G$1" x="83.82" y="132.08"/>
-<instance part="C3" gate="G$1" x="121.92" y="99.06"/>
-<instance part="Q1" gate="G$1" x="121.92" y="81.28"/>
+<instance part="C3" gate="G$1" x="121.92" y="55.88"/>
 <instance part="U$1" gate="J" x="50.8" y="38.1" rot="R180"/>
 <instance part="S2" gate="G$1" x="83.82" y="91.44"/>
-<instance part="LEDPWR" gate="G$1" x="109.22" y="101.6" rot="MR180"/>
+<instance part="LEDPWR" gate="G$1" x="109.22" y="58.42" rot="MR180"/>
 <instance part="LEDSIG" gate="G$1" x="81.28" y="71.12" rot="MR0"/>
 <instance part="LED1" gate="G$1" x="27.94" y="134.62" rot="MR0"/>
@@
 <instance part="R3" gate="G$1" x="40.64" y="124.46" rot="R90"/>
 <instance part="SUPPLY7" gate="P" x="55.88" y="27.94" rot="R180"/>
-<instance part="SUPPLY11" gate="P" x="121.92" y="111.76"/>
+<instance part="SUPPLY11" gate="P" x="157.48" y="83.82"/>
 <instance part="SUPPLY12" gate="P" x="15.24" y="91.44"/>
 <instance part="SUPPLY13" gate="P" x="83.82" y="147.32"/>
@@
 <instance part="FRAME1" gate="G$1" x="0" y="0"/>
 <instance part="FRAME1" gate="G$2" x="147.32" y="0"/>
-<instance part="R4" gate="G$1" x="106.68" y="81.28"/>
+<instance part="LEDSW" gate="G$1" x="139.7" y="77.47"/>
+<instance part="SUPPLY3" gate="GND" x="139.7" y="63.5"/>
+<instance part="C4" gate="G$1" x="157.48" y="72.39"/>
+<instance part="SUPPLY4" gate="GND" x="157.48" y="63.5"/>
+<instance part="C5" gate="G$1" x="127" y="72.39"/>
+<instance part="SUPPLY14" gate="GND" x="127" y="67.31"/>
 </instances>
 <busses>
@@
 </segment>
 <segment>
+<pinref part="C3" gate="G$1" pin="2"/>
+<pinref part="LEDPWR" gate="G$1" pin="2"/>
+<wire x1="116.84" y1="55.88" x2="116.84" y2="53.34" width="0.1524" layer="91"/>
+<wire x1="116.84" y1="53.34" x2="121.92" y2="53.34" width="0.1524" layer="91"/>
 <pinref part="SUPPLY5" gate="GND" pin="GND"/>
-<pinref part="Q1" gate="G$1" pin="S"/>
-<wire x1="121.92" y1="73.66" x2="121.92" y2="76.2" width="0.1524" layer="91"/>
+<wire x1="121.92" y1="53.34" x2="121.92" y2="43.18" width="0.1524" layer="91"/>
+<junction x="121.92" y="53.34"/>
+</segment>
+<segment>
+<pinref part="LEDSW" gate="G$1" pin="GND"/>
+<pinref part="SUPPLY3" gate="GND" pin="GND"/>
+<wire x1="139.7" y1="67.31" x2="139.7" y2="66.04" width="0.1524" layer="91"/>
+</segment>
+<segment>
+<pinref part="C4" gate="G$1" pin="2"/>
+<pinref part="SUPPLY4" gate="GND" pin="GND"/>
+<wire x1="157.48" y1="69.85" x2="157.48" y2="66.04" width="0.1524" layer="91"/>
+</segment>
+<segment>
+<pinref part="C5" gate="G$1" pin="2"/>
+<pinref part="SUPPLY14" gate="GND" pin="GND"/>
 </segment>
 </net>
@@
 <segment>
 <pinref part="ATTINY85" gate="G$1" pin="PB2(SCK/ADC1)"/>
-<wire x1="53.34" y1="81.28" x2="101.6" y2="81.28" width="0.1524" layer="91"/>
-<pinref part="R4" gate="G$1" pin="1"/>
+<wire x1="53.34" y1="81.28" x2="128.27" y2="81.28" width="0.1524" layer="91"/>
+<pinref part="LEDSW" gate="G$1" pin="IN"/>
 </segment>
 </net>
@@
 <label x="58.42" y="71.12" size="1.016" layer="95" rot="R270" xref="yes"/>
 </segment>
-<segment>
-<pinref part="CHARGE" gate="G$1" pin="STAT"/>
-<pinref part="LED2" gate="G$1" pin="A"/>
-<wire x1="40.64" y1="137.16" x2="45.72" y2="137.16" width="0.1524" layer="91"/>
-<wire x1="40.64" y1="137.16" x2="40.64" y2="149.86" width="0.1524" layer="91"/>
-<junction x="40.64" y="137.16"/>
-<label x="40.64" y="149.86" size="1.016" layer="95" rot="R90" xref="yes"/>
-</segment>
 </net>
 <net name="+4.1V" class="1">
@@
 </segment>
 <segment>
+<pinref part="SUPPLY11" gate="P" pin="+4.1V"/>
+<pinref part="LEDSW" gate="G$1" pin="FB"/>
+<wire x1="151.13" y1="77.47" x2="157.48" y2="77.47" width="0.1524" layer="91"/>
+<wire x1="157.48" y1="77.47" x2="157.48" y2="81.28" width="0.1524" layer="91"/>
+<pinref part="C4" gate="G$1" pin="1"/>
+<junction x="157.48" y="77.47"/>
+</segment>
+</net>
+<net name="N$6" class="1">
+<segment>
 <pinref part="C3" gate="G$1" pin="1"/>
 <pinref part="LEDPWR" gate="G$1" pin="1"/>
-<wire x1="116.84" y1="101.6" x2="116.84" y2="104.14" width="0.1524" layer="91"/>
-<wire x1="116.84" y1="104.14" x2="121.92" y2="104.14" width="0.1524" layer="91"/>
-<pinref part="SUPPLY11" gate="P" pin="+4.1V"/>
-<wire x1="121.92" y1="109.22" x2="121.92" y2="104.14" width="0.1524" layer="91"/>
-<junction x="121.92" y="104.14"/>
-</segment>
-</net>
-<net name="N$2" class="1">
-<segment>
-<pinref part="C3" gate="G$1" pin="2"/>
-<pinref part="LEDPWR" gate="G$1" pin="2"/>
-<wire x1="116.84" y1="99.06" x2="116.84" y2="96.52" width="0.1524" layer="91"/>
-<wire x1="116.84" y1="96.52" x2="121.92" y2="96.52" width="0.1524" layer="91"/>
-<pinref part="Q1" gate="G$1" pin="D"/>
-<wire x1="121.92" y1="96.52" x2="121.92" y2="86.36" width="0.1524" layer="91"/>
-<junction x="121.92" y="96.52"/>
-</segment>
-</net>
-<net name="N$1" class="0">
-<segment>
-<pinref part="R4" gate="G$1" pin="2"/>
-<pinref part="Q1" gate="G$1" pin="G"/>
-<wire x1="111.76" y1="81.28" x2="114.3" y2="81.28" width="0.1524" layer="91"/>
-</segment>
-</net>
+<wire x1="116.84" y1="58.42" x2="116.84" y2="60.96" width="0.1524" layer="91"/>
+<wire x1="116.84" y1="60.96" x2="121.92" y2="60.96" width="0.1524" layer="91"/>
+<junction x="121.92" y="60.96"/>
+<pinref part="LEDSW" gate="G$1" pin="EN"/>
+<wire x1="128.27" y1="77.47" x2="127" y2="77.47" width="0.1524" layer="91"/>
+<wire x1="127" y1="77.47" x2="121.92" y2="77.47" width="0.1524" layer="91"/>
+<wire x1="121.92" y1="77.47" x2="121.92" y2="60.96" width="0.1524" layer="91"/>
+<pinref part="C5" gate="G$1" pin="1"/>
+<junction x="127" y="77.47"/>
+</segment>
+</net>
+<net name="STAT" class="0">
+<segment>
+<pinref part="CHARGE" gate="G$1" pin="STAT"/>
+<pinref part="LED2" gate="G$1" pin="A"/>
+<wire x1="40.64" y1="137.16" x2="45.72" y2="137.16" width="0.1524" layer="91"/>
+</segment>
+</net>
